Commit message: update bimanual

File: bimanual/rtop_description/urdf/rtop.urdf (robot description, URDF)
Before this commit: robot rtop, 49 links, 48 joints
Links:
- link base: geometry collision box size=0.30 1.0 0.25; collision box size=0.8 0.12 0.10

File: bimanual/rtop_description/urdf/rtop.urdf.xacro (robot description, xacro)
@@ -10,14 +10,43 @@
       <inertia ixx="1.0" iyy="1.0" izz="1.0" ixy="0" ixz="0" iyz="0"/>
     </inertial>
+    <!-- TRONCO -->
     <visual name="base_visual">
-      <origin xyz="0.0 0.0 0.0" rpy="1.5708 0.0 1.5708"/>
+      <origin xyz="0.0 0.0 1.0" rpy="1.5708 0.0 1.5708"/>
       <geometry>
-        <mesh filename="package://rtop_description/meshes/body.obj"/>
+        <box size="0.30 1.0 0.25"/>
+      </geometry>
+    </visual>
+    <!-- HOMBROS -->
+    <visual name="base_visual_hombros">
+      <origin xyz="0.0 0.0 1.0" rpy="1.5708 0.0 1.5708"/>
+      <geometry>
+        <box size="0.8 0.12 0.10"/>
+      </geometry>
+    </visual>
+    <!-- CABEZA -->
+    <visual name="base_visual_cabeza">
+      <origin xyz="0.0 0.0 1.65" rpy="1.5708 0.0 1.5708"/>
+      <geometry>
+        <sphere radius="0.125"/>
       </geometry>
     </visual>
     <collision name="base_collision">
-      <origin xyz="0.0 0.0 0.0" rpy="1.5708 0.0 1.5708"/>
+      <origin xyz="0.0 0.0 1.0" rpy="1.5708 0.0 1.5708"/>
       <geometry>
-        <mesh filename="package://rtop_description/meshes/body.obj"/>
+        <box size="0.30 1.0 0.25"/>
+      </geometry>
+    </collision>
+    <!-- HOMBROS -->
+    <collision name="base_collision_hombros">
+      <origin xyz="0.0 0.0 1.0" rpy="1.5708 0.0 1.5708"/>
+      <geometry>
+        <box size="0.8 0.12 0.10"/>
+      </geometry>
+    </collision>
+    <!-- CABEZA -->
+    <collision name="base_collision_cabeza">
+      <origin xyz="0.0 0.0 1.65" rpy="1.5708 0.0 1.5708"/>
+      <geometry>
+        <sphere radius="0.125"/>
       </geometry>
     </collision>

File: single/yam_arm_description/urdf/yam_arm_gazebo.urdf.xacro (robot description, xacro)
@@ -3,7 +3,7 @@
   <!-- Arguments -->
   <xacro:arg name="use_gazebo" default="true"/>
-  <xacro:arg name="ros2_controllers_path" default="yam_arm_description/config/ros2_controllers.yaml"/>
+  <xacro:arg name="ros2_controllers_path" default="yam_arm_moveit_config/config/ros2_controllers.yaml"/>
   <!-- Include the base robot description as xacro -->
-  <xacro:include filename="$(find yam_arm_description)/urdf/yam_arm_gazebo_macro.xacro"/>
+  <xacro:include filename="$(find yam_arm_description)/urdf/yam_arm_macro.xacro"/>
    <!-- World link -->
    <link name="world">
